File: hardware/board/mainboard.kicad_pcb (KiCad board)
At the start: 4 copper layers, 60 x 110 mm, 279 parts, among them J201 Power, Q601 BCM847, Q701 BCM847, Q801 BCM847, Q901 MMBT3906, U1 TL074, U2 TL074, U201 TL431A, U3 TL074, U4 TL074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

Commit message: Remove logo; Add Sherpa Modular manufacturing note
Parts:
- removed the ? at (80.7, 144.8)
- removed the G*** at (79.1, 134.0)
Other:
- rule pad_to_mask_clearance: 0.0381 -> 0
- board text added: "Manufactured by Sherpa Modular 2025-10-29"
